File: hardware/ESP32-S3 Parallel TFT with Touch 4.3“ V1.3.brd (EAGLE design)
At the start: 67.2 x 117.6 mm, 100 parts, among them IC1 CP2104, P2 AFC01-S06FCC-00, P5 FPC-40P, Q1 32.768K, Q2 AO3400, Q3 S8050, Q4 S8050, Q5 MOSFET-PCHANNEL, U1 ESP32­S2­SOLO, U2 RY3730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

Commit message: V1.3 hardware update
Parts:
- added R34, R38, R40: NC, Discrete:R0603
- added R35: 0R, Discrete:R0603
- added R36, R37, R39: NC, A9G:DISCRETE_R0603
- C13: value 0.1uF -> NC
- R27: value 10K -> NC
- R32: value 50R -> 12R
- R33: value 50R -> NC
- moved BT1 70.3 mm to (14.8, 11.0), turned to 0 degrees
- moved U$1 42.4 mm to (7.94, 61.5)
- moved R24 34.6 mm to (42.6, 93.2), turned to 180 degrees
- moved R17 34.4 mm to (50.2, 93.0), turned to 90 degrees
- moved Q5 34.1 mm to (45.9, 93.2)
- moved D5 33.9 mm to (48.5, 93.4)
- moved C14 31.5 mm to (51.9, 102.9)
- moved C25 31.2 mm to (49.2, 96.2), turned to 180 degrees
- moved R2 29.4 mm to (46.0, 96.2), turned to 0 degrees
- moved C15 24.3 mm to (42.6, 94.7), turned to 0 degrees
- moved C17 22.4 mm to (42.6, 96.2), turned to 0 degrees
- moved U3 22.2 mm to (46.8, 100.2), turned to 0 degrees
- moved C18 21.3 mm to (41.4, 102.9), turned to 90 degrees
- moved C54 20.5 mm to (55.0, 17.9), turned to 90 degrees
- moved R28 20.1 mm to (41.3, 43.8), turned to 0 degrees
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Connections:
- removed net IO38/INT: P2.4, U1.31, U8.7
- new net IO38: R35.1, R38.1, U1.31, U8.7
- new net TP_INT: P2.4, R36.1, R37.1, R38.2
- net 3.3V: now also R36.2
- net 5V: now also R39.2
- net GND: now also R37.2
- net IO2/BLK: now also R40.1
- net N$24: now also R39.1
- net RESET: now also R34.1
- net RST: now also R34.2, R35.2, R40.2
Routing:
- net N$20: track 6.11 -> 127.1 mm, vias 0 -> 2
- net IO38: track 0.00 -> 58.9 mm, vias 0 -> 3
- net IO38/INT: track 44.6 -> 0.00 mm, vias 3 -> 0
- net 3.3V: track 128.8 -> 172.0 mm, vias 5 -> 6
- net IO2/BLK: track 20.4 -> 61.2 mm, vias 2 -> 3
- net N$17: track 42.7 -> 8.20 mm
- net RST: track 21.3 -> 42.6 mm
- net +3V3: track 231.4 -> 252.7 mm
- net TXD/IO43: track 30.7 -> 51.9 mm
- net IO13/MISO: track 62.4 -> 78.8 mm
- net IO10/CS: track 47.8 -> 64.1 mm
- net IO11/MOSI: track 47.2 -> 63.3 mm
- net LED-: track 38.6 -> 54.6 mm
- net IO12/SCLK: track 51.6 -> 67.2 mm
- net RESET: track 65.8 -> 81.1 mm
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- added copper zone on layer 1, net N$17
- removed copper zone on layer 1, net +3V3
- removed copper zone on layer 1, net 3.3V
- removed copper zone on layer 1, net VBUS
Other:
- outline, holes or cut-outs redrawn
- board text added: "IO17/SDA"
- board text added: "IO18/SCL"
- board text added: "IO19/D-"
- board text added: "IO20/D+"
- board text added: "with Touch 4.3" V1.3"
- board text removed: "D+"
- board text removed: "D-"
- board text removed: "IO17"
- board text removed: "IO18"
- board text removed: "IO19"
- board text removed: "IO20"
- board text removed: "SCL"
- board text removed: "SDA"
- board text removed: "with Touch 4.3" V1.1"
