File: hardware/ESP32-S3 Parallel TFT with Touch 4.3“ V1.3.sch (EAGLE design)
At the start: 99 parts, among them IC1 CP2104, P2 AFC01-S06FCC-00, P5 FPC-40P, Q1 32.768K, Q2 AO3400, Q3 S8050, Q4 S8050, Q5 MOSFET-PCHANNEL, U1 ESP32­S2­SOLO, U2 RY3730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

Commit message: V1.3 hardware update
Parts:
- added R34, R38, R40: NC, Discrete:R-0603
- added R35: 0R, Discrete:R-0603
- added R36, R37, R39: NC, A9G:DISCRETE_R-0603
- C13: value 0.1uF -> NC
- R27: value 10K -> NC
- R32: value 50R -> 12R
- R33: value 50R -> NC
Connections:
- removed net IO38/INT: P2.4, U1.IO38, U8.PENIRQ
- new net IO38: R35.1, R38.1, U1.IO38, U8.PENIRQ
- new net TP_INT: P2.4, R36.1, R37.1, R38.2
- net 3.3V: now also R36.2
- net 5V: now also R39.2
- net GND: now also R37.2
- net IO2/BLK: now also R40.1
- net N$24: now also R39.1
- net RESET: now also R34.1
- net RST: now also R34.2, R35.2, R40.2
Other:
- note added: "ESP32-S3 Parallel TFT with Touch 4.3“ V1.3"
- note removed: "ESP32-S3 Parallel TFT with Touch 4.3“ V1.1"
- moved on the sheet: R28
