File: hardware/ESP32-S3 Parallel TFT with Touch 4.3“ V2.0.brd (EAGLE design)
At the start: 67.2 x 117.6 mm, 107 parts, among them IC1 CP2104, P2 AFC01-S06FCC-00, P5 FPC-40P, Q1 32.768K, Q2 AO3400, Q3 S8050, Q4 S8050, Q5 MOSFET-PCHANNEL, U1 ESP32­S2­SOLO, U2 RY3730, U3 PCF8563T/5,518, U4 LD1117/3.3v, U8 NS2009

Commit message: V2.0 Hardware
Parts:
- removed C16: 4.7uF/16V, Discrete:0603
- removed R1: 0R, Discrete:R0603
- removed R40: NC, Discrete:R0603
- removed U4: LD1117/3.3v, IC:SOT89
- added BAT: JST-2P, Connector-new:HW2-SMD-2.0-90D
- added C26, C27, C37, C39: 0.1uF, Discrete:0603
- added C28, C35, C36, C38, C40, C42: 10uF, Discrete:0603
- added C33, C34: 50pF, Discrete:0603
- added C41: 4.7uF/16V, Discrete:0603
- added C45: NC, Discrete:0603
- added CHRG: RED, microbuilder:CHIPLED_0805_NOOUTLINE
- added D11, D3: B5819WS, Discrete:SOD323
- added DONE: GREEN, microbuilder:CHIPLED_0805_NOOUTLINE
- added IC2: MAX98357A, SparkFun-IC-Amplifiers:TQFN-16
- added Q6: MOSFET-PCHANNEL, User-Submitted:SOT23-3
- added Q7: S8050, Discrete:SOT23
- added R41, R43, R48, R51, R53, R54, R63: 0R, Discrete:R0603
- added R46, R56, R57: NC, Discrete:R0603
- added R55: 560K, Discrete:R0603
- added R58: 100k, Discrete:R0603
- added R59: NC, A9G:DISCRETE_R0603
- added R60: 10K, A9G:DISCRETE_R0603
- added R61, R62: 1.2K, Discrete:R0603
- added SPK: 1X2P, sale:1X2P-SMT1.25MM
- added U5: SPX3819, IC:SOT23-5
- added U6: TP4056, self:SOP8-1.27P
- C2: value 100pF/50V -> 10pF/50V
- R19: value 470R -> 1.2K
- R23: value 100R -> 50R
- R24: value 50R -> 12R
- R28: value 100R -> 1.2K; device A9G:DISCRETE_R0603 -> Discrete:R0603
- R31: value 10K -> NC
- R39: value NC -> 10K
- moved C14 35.5 mm to (16.5, 100.6), turned to 0 degrees
- moved R17 34.2 mm to (16.6, 86.9), turned to 0 degrees
- moved Q5 32.8 mm to (13.3, 89.5)
- moved D5 32.8 mm to (15.9, 89.6)
- moved C25 32.8 mm to (16.7, 92.3)
- moved R2 32.7 mm to (13.5, 92.3)
- moved C17 32.7 mm to (10.1, 92.5)
- moved C15 32.7 mm to (10.1, 91.0)
- moved R24 32.7 mm to (10.1, 89.5)
- moved U3 32.5 mm to (14.5, 96.5)
- moved J2 32.2 mm to (25.5, 95.7), turned to 0 degrees
- moved C18 31.8 mm to (9.80, 99.2)
- moved C19 31.8 mm to (9.80, 96.2)
- moved Q1 31.6 mm to (7.75, 97.7)
- moved R28 29.6 mm to (49.5, 72.2), turned to 180 degrees
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Connections:
- removed net IO2/BLK: R28.2, R40.1, U1.38
- new net !SD: IC2.P$4, R55.1
- new net GAIN: IC2.P$2, R56.1, R57.2
- new net I2S_BCLK: IC2.P$16, R53.2
- new net I2S_DIN: IC2.P$1, R51.2
- new net I2S_LRCLK: IC2.P$14, R54.2
- new net IO2: R54.1, U1.38
- new net N$21: IC2.P$9, R41.1
- new net N$23: IC2.P$10, R43.1
- new net N$26: C33.2, R41.2, SPK.1
- new net N$27: C34.2, R43.2, SPK.2
- new net N$29: Q7.1, R59.1, R60.2
- new net N$30: R28.1, U6.2
- new net N$31: R61.2, U6.7
- new net N$32: R62.2, U6.6
- new net N$33: CHRG.C, R61.1
- new net N$34: DONE.C, R62.1
- new net N$76: C45.1, U5.4
- new net VBAT: BAT.+, C40.1, D11.+, Q6.3, U6.5
- new net VDD: C26.2, C27.2, C28.2, IC2.P$7, IC2.P$8, R46.1, R48.1, R55.2, R56.2
- new net VPWR: C35.2, C41.1, D11.-, D3.-, L1.P$1, Q6.2, R39.2, R48.2, U2.6, U5.1, U5.3
- net +3V3: now also C42.1, R46.2, R63.1, U5.5; no longer C22.1, R1.1, U4.2, U4.4
- net 3.3V: now also C22.1, R63.2; no longer R1.2
- net 5V: now also C36.2, C37.1, C38.1, C39.1, CHRG.A, D3.+, DONE.A, Q6.1, R58.1, U6.4, U6.8; no longer C16.1, L1.P$1, R39.2, U2.6, U4.3
- net GND: now also BAT.-, BAT.3, BAT.4, C26.1, C27.1, C28.1, C33.1, C34.1, C35.1, C36.1, C37.2, C38.2, C39.2, C40.2, C41.2, C42.2, C45.2, IC2.P$11, IC2.P$15, IC2.P$3, IC2.P$EP, Q7.2, R28.2, R57.1, R58.2, R60.1, SPK.3, SPK.4, U5.2, U6.1, U6.3, U6.9; no longer C16.2, U4.1
- net IO19: now also R51.1
- net IO20: now also R53.1
- net N$24: now also Q7.3; no longer R28.1
- net RST: no longer R40.2
- net RXD/IO44: now also R59.2
Routing:
- net IO2: track 0.00 -> 89.5 mm, vias 0 -> 2
- net IO2/BLK: track 61.2 -> 0.00 mm, vias 3 -> 0
- net VPWR: track 0.00 -> 53.9 mm
- net +3V3: track 252.7 -> 215.3 mm, vias 8 -> 9
- net IO18/I2C_SCL: track 151.5 -> 116.1 mm
- net N$20: track 127.1 -> 93.3 mm
- net IO20: track 68.3 -> 101.7 mm, vias 2 -> 4
- net IO17/I2C_SDA: track 142.4 -> 111.0 mm
- net IO19: track 74.3 -> 105.6 mm, vias 2 -> 3
- net 3.3V: track 172.0 -> 141.7 mm
- net N$32: track 0.00 -> 19.3 mm, vias 0 -> 2
- net VDD: track 0.00 -> 19.2 mm
- net 5V: track 58.5 -> 74.7 mm, vias 4 -> 6
- net N$31: track 0.00 -> 15.0 mm, vias 0 -> 2
- net N$12: track 14.0 -> 3.95 mm
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- added copper zone on layer 1, net +3V3
- added copper zone on layer 1, net 3.3V
- added copper zone on layer 1, net VBAT
- added copper zone on layer 1, net VDD
- added copper zone on layer 1, net VPWR
- added copper zone on layer 1, net VRTC
Other:
- board text added: "with Touch 4.3" V2.0"
- board text removed: "with Touch 4.3" V1.3"
