File: hardware/ESP32-S3 Parallel TFT with Touch 4.3“ V2.0.sch (EAGLE design)
At the start: 106 parts, among them IC1 CP2104, P2 AFC01-S06FCC-00, P5 FPC-40P, Q1 32.768K, Q2 AO3400, Q3 S8050, Q4 S8050, Q5 MOSFET-PCHANNEL, U1 ESP32­S2­SOLO, U2 RY3730, U3 PCF8563T/5,518, U4 LD1117/3.3v, U8 NS2009

Commit message: V2.0 Hardware
Parts:
- removed C16: 4.7uF/16V, Discrete:C-0603
- removed R1: 0R, Discrete:R-0603
- removed R40: NC, Discrete:R-0603
- removed U4: LD1117/3.3v, IC:LD1117'SOT89'
- added BAT: JST-2P, Connector-new:JST-2P-SMD'2.0'
- added C26, C27, C37, C39: 0.1uF, Discrete:C-0603
- added C28, C35, C36, C38, C40, C42: 10uF, Discrete:C-0603
- added C33, C34: 50pF, Discrete:C-0603
- added C41: 4.7uF/16V, Discrete:C-0603
- added C45: NC, Discrete:C-0603
- added CHRG: RED, microbuilder:LED0805_NOOUTLINE
- added D11, D3: B5819WS, Discrete:D'0805'
- added DONE: GREEN, microbuilder:LED0805_NOOUTLINE
- added IC2: MAX98357A, SparkFun-IC-Amplifiers:MAX98357A
- added Q6: MOSFET-PCHANNEL, User-Submitted:MOSFET-PCHANNEL
- added Q7: S8050, Discrete:TRANSISTOR-NPN-SOT23
- added R41, R43, R48, R51, R53, R54, R63: 0R, Discrete:R-0603
- added R46, R56, R57: NC, Discrete:R-0603
- added R55: 560K, Discrete:R-0603
- added R58: 100k, Discrete:R-0603
- added R59: NC, A9G:DISCRETE_R-0603
- added R60: 10K, A9G:DISCRETE_R-0603
- added R61, R62: 1.2K, Discrete:R-0603
- added SPK: 1X2P, sale:1X2P
- added U5: SPX3819, IC:SPX3819
- added U6: TP4056, self:TP4056
- C2: value 100pF/50V -> 10pF/50V
- R19: value 470R -> 1.2K
- R23: value 100R -> 50R
- R24: value 50R -> 12R
- R28: value 100R -> 1.2K; device A9G:DISCRETE_R-0603 -> Discrete:R-0603
- R31: value 10K -> NC
- R39: value NC -> 10K
Connections:
- removed net IO2/BLK: R28.2, R40.1, U1.IO2
- new net !SD: IC2.!SD_MODE, R55.1
- new net GAIN: IC2.GAIN, R56.1, R57.2
- new net I2S_BCLK: IC2.BCLK, R53.2
- new net I2S_DIN: IC2.DIN, R51.2
- new net I2S_LRCLK: IC2.LRCLK, R54.2
- new net IO2: R54.1, U1.IO2
- new net N$21: IC2.OUT+, R41.1
- new net N$23: IC2.OUT-, R43.1
- new net N$26: C33.2, R41.2, SPK.1
- new net N$27: C34.2, R43.2, SPK.2
- new net N$29: Q7.B, R59.1, R60.2
- new net N$30: R28.1, U6.ISET
- new net N$31: R61.2, U6.CHRG
- new net N$32: R62.2, U6.DONE
- new net N$33: CHRG.C, R61.1
- new net N$34: DONE.C, R62.1
- new net N$76: C45.1, U5.BYP
- new net VBAT: BAT.1, C40.1, D11.+, Q6.D, U6.BAT
- new net VDD: C26.2, C27.2, C28.2, IC2.VDD, R46.1, R48.1, R55.2, R56.2
- new net VPWR: C35.2, C41.1, D11.-, D3.-, L1.1, Q6.S, R39.2, R48.2, U2.IN, U5.EN, U5.VIN
- net +3V3: now also C42.1, R46.2, R63.1, U5.VOUT; no longer C22.1, R1.1, U4.OUT
- net 3.3V: now also C22.1, R63.2; no longer R1.2
- net 5V: now also C36.2, C37.1, C38.1, C39.1, CHRG.A, D3.+, DONE.A, Q6.G, R58.1, U6.CE, U6.VIN; no longer C16.1, L1.1, R39.2, U2.IN, U4.IN
- net GND: now also BAT.2, BAT.3, BAT.4, C26.1, C27.1, C28.1, C33.1, C34.1, C35.1, C36.1, C37.2, C38.2, C39.2, C40.2, C41.2, C42.2, C45.2, IC2.GND, Q7.E, R28.2, R57.1, R58.2, R60.1, SPK.3, SPK.4, U5.GND, U6.GND, U6.GND@1, U6.TEMP; no longer C16.2, U4.GND
- net IO19: now also R51.1
- net IO20: now also R53.1
- net N$24: now also Q7.C; no longer R28.1
- net RST: no longer R40.2
- net RXD/IO44: now also R59.2
Other:
- note added: "0.16V"
- note added: "0.5V"
- note added: "0.77V"
- note added: "1.4V"
- note added: "100K"
- note added: "9dB"
- note added: "ESP32-S3 Parallel TFT with Touch 4.3“ V2.0"
- note added: "LDO&Charger"
- note added: "LEFT"
- note added: "LEFT/2 + RIGHT/2"
- note added: "ME6217"
- note added: "RIGHT"
- note added: "VDD: 2.5-5.5V"
- note added: "Voltage of !SD"
- note removed: "ESP32-S3 Parallel TFT with Touch 4.3“ V1.3"
- moved on the sheet: C22, R28
