File: hardware/ESP32-S3 Parallel TFT with Touch 4.3“ V3.1.brd (EAGLE design)
At the start: 67.2 x 117.6 mm, 144 parts, among them IC1 CP2104, IC2 MAX98357A, P2 AFC01-S06FCC-00, P5 FPC-40P, Q1 32.768K, Q2 AO3400, Q3 S8050, Q4 S8050, Q5 MOSFET-PCHANNEL, Q6 MOSFET-PCHANNEL, Q7 S8050, U1 ESP32­S2­SOLO, U2 RY3730, U3 PCF8563T/5,518, U5 SPX3819, U6 TP4056, U8 NS2009

Commit message: Update hardware
Parts:
- removed BT1: CR2032, sale:CR2032
- removed C14, C15, C30, C32: 0.1uF, A9G:DISCRETE_C0603
- removed C17, C29, C31: 10uF, A9G:DISCRETE_C0603
- removed C18, C19: 20pF, A9G:DISCRETE_C0603
- removed C25: 10uF, Discrete:0603
- removed D2: 1N4148WS, Discrete:SOD323
- removed FLASH: BUTTON, MySMD:157SW
- removed LED1: NC, Relay:DISCRETE_LED-3528
- removed Q1: 32.768K, microbuilder:XTAL3215
- removed Q2: AO3400, Discrete:SOT23@1
- removed Q5: MOSFET-PCHANNEL, User-Submitted:SOT23-3
- removed R17, R45: 100k, Discrete:R0603
- removed R18: 10R, A9G:DISCRETE_R0603
- removed R2: 50R, Discrete:R0603
- removed R24: 12R, Discrete:R0603
- removed R49: 0R, A9G:DISCRETE_R0603
- removed R50: NC, Discrete:R0603
- removed R52: NC, A9G:DISCRETE_R0603
- removed U3: PCF8563T/5,518, sale:SOP8
- removed U8: NS2009, NS2009:MSOP10
- added BOOT: TS24CA, sale:2*4*3.5MM
- added M1, M2, M3, M4, M5, M6, M7, M8: M2.5, sale:M2.5
- D3: value B5819WS -> SS54; device Discrete:SOD323 -> diode:DO-214AC
- D5: value 1N4148WS -> SS54; device Discrete:SOD323 -> diode:DO-214AC
- R32: value 12R -> 3R3
- R57: value NC -> 10K
- RST: value BUTTON -> TS24CA; device MySMD:157SW -> sale:2*4*3.5MM
- moved D5 45.7 mm to (52.7, 62.4), turned to 270 degrees
- moved R63 28.4 mm to (9.55, 24.8), turned to 0 degrees
- moved R27 27.5 mm to (9.55, 23.3), turned to 180 degrees
- moved C23 27.4 mm to (18.5, 28.7), turned to 270 degrees
- moved R44 27.3 mm to (14.6, 28.0), turned to 180 degrees
- moved C13 27.2 mm to (17.0, 28.8), turned to 270 degrees
- moved C22 26.1 mm to (13.1, 26.4), turned to 180 degrees
- moved R42 25.7 mm to (12.1, 24.0), turned to 90 degrees
- moved SD 25.1 mm to (22.2, 15.1)
- moved R47 23.1 mm to (13.7, 24.0), turned to 90 degrees
- moved R29 19.6 mm to (39.8, 45.4), turned to 0 degrees
- moved D3 18.2 mm to (43.1, 63.2), turned to 0 degrees
- moved C36 17.0 mm to (47.1, 64.0), turned to 90 degrees
- moved C24 16.7 mm to (20.1, 28.8), turned to 270 degrees
- moved R58 14.6 mm to (48.6, 79.4)
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Connections:
- removed net N$13: C19.1, Q1.P$2, U3.2
- removed net N$15: Q5.3, R24.1
- removed net N$16: C15.2, C17.2, R2.1
- removed net N$20: BT1.2, R24.2
- removed net N$25: R49.2, R52.1, U8.8
- removed net N$4: C18.1, Q1.P$1, U3.1
- removed net N$5: Q2.1, R45.2, R50.1
- removed net N$8: LED1.1, R18.1
- removed net N$9: LED1.2, Q2.3
- removed net VRTC: C14.2, C25.2, D5.-, Q5.2, R2.2, U3.8
- net 3.3V: no longer C29.2, C30.2, C31.1, C32.1, D5.+, Q5.1, R17.1, R52.2, U8.1
- net 5V: now also D3.A, D5.C; no longer D2.-, D3.+, R18.2
- net GND: now also BOOT.1, BOOT.3, BOOT.4, M1.1, M2.1, M3.1, M4.1, M5.1, M6.1, M7.1, M8.1, RST.3, RST.4; no longer BT1.1, C14.1, C15.1, C17.1, C18.2, C19.2, C25.1, C29.1, C30.1, C31.2, C32.2, FLASH.1, Q2.2, R17.2, R45.1, R49.1, U3.4, U8.6
- net IO0: now also BOOT.2; no longer FLASH.2
- net IO17/I2C_SDA: no longer U3.5, U8.9
- net IO18/I2C_SCL: no longer U3.6, U8.10
- net IO38: no longer U8.7
- net TXD/IO43: no longer R50.2
- net VBUS: now also D5.A; no longer D2.+
- net VPWR: now also D3.C; no longer D3.-
- net XN: no longer U8.4
- net XP: no longer U8.2
- net YN: no longer U8.5
- net YP: no longer U8.3
Routing:
- net N$20: track 93.3 -> 0.00 mm, vias 2 -> 0
- net GND: track 38.9 -> 125.4 mm, vias 400 -> 212
- net +3V3: track 215.3 -> 291.8 mm, vias 9 -> 7
- net XP: track 68.3 -> 0.00 mm, vias 2 -> 0
- net YP: track 67.0 -> 0.00 mm, vias 2 -> 0
- net XN: track 65.8 -> 0.00 mm, vias 2 -> 0
- net YN: track 64.5 -> 0.00 mm, vias 2 -> 0
- net 3.3V: track 141.7 -> 97.6 mm, vias 6 -> 3
- net RST: track 40.8 -> 10.5 mm, vias 2 -> 0
- net IO18/I2C_SCL: track 116.1 -> 89.1 mm
- net RXD/IO44: track 60.0 -> 34.5 mm, vias 4 -> 2
- net IO38: track 58.9 -> 33.4 mm, vias 3 -> 2
- net IO17/I2C_SDA: track 111.0 -> 86.9 mm
- net N$48: track 2.40 -> 24.6 mm
- net IO12/SCLK: track 67.2 -> 85.1 mm, vias 2 -> 3
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- removed copper zone on layer 1, net +3V3
- removed copper zone on layer 1, net 3.3V
- removed copper zone on layer 1, net 5V
- removed copper zone on layer 1, net N$17
- removed copper zone on layer 1, net VRTC
Other:
- board size 67.2 x 117.6 mm -> 67.2 x 105.5 mm
- board text added: "with Touch 4.3" V3.1"
- board text removed: "with Touch 4.3" V2.0"
