File: hardware/ESP32-S3 Parallel TFT with Touch 4.3“ V3.1.sch (EAGLE design)
At the start: 143 parts, among them IC1 CP2104, IC2 MAX98357A, P2 AFC01-S06FCC-00, P5 FPC-40P, Q1 32.768K, Q2 AO3400, Q3 S8050, Q4 S8050, Q5 MOSFET-PCHANNEL, Q6 MOSFET-PCHANNEL, Q7 S8050, U1 ESP32­S2­SOLO, U2 RY3730, U3 PCF8563T/5,518, U5 SPX3819, U6 TP4056, U8 NS2009

Commit message: Update hardware
Parts:
- removed BT1: CR2032, sale:CR2032
- removed C14, C15, C30, C32: 0.1uF, A9G:DISCRETE_C-0603
- removed C17, C29, C31: 10uF, A9G:DISCRETE_C-0603
- removed C18, C19: 20pF, A9G:DISCRETE_C-0603
- removed C25: 10uF, Discrete:C-0603
- removed D2: 1N4148WS, Discrete:D'0805'
- removed FLASH: BUTTON, MySMD:PB157
- removed LED1: NC, Relay:DISCRETE_LED3528
- removed Q1: 32.768K, microbuilder:CRYSTAL_3215
- removed Q2: AO3400, Discrete:MOSFET-N'SOT23'
- removed Q5: MOSFET-PCHANNEL, User-Submitted:MOSFET-PCHANNEL
- removed R17, R45: 100k, Discrete:R-0603
- removed R18: 10R, A9G:DISCRETE_R-0603
- removed R2: 50R, Discrete:R-0603
- removed R24: 12R, Discrete:R-0603
- removed R49: 0R, A9G:DISCRETE_R-0603
- removed R50: NC, Discrete:R-0603
- removed R52: NC, A9G:DISCRETE_R-0603
- removed U3: PCF8563T/5,518, sale:PCF8563T/5,518
- removed U8: NS2009, NS2009:NS2009
- added BOOT: TS24CA, sale:TS24CA
- added M1, M2, M3, M4, M5, M6, M7, M8: M2.5, sale:M2.5
- D3: value B5819WS -> SS54; device Discrete:D'0805' -> diode:DIODE-DO-214AC
- D5: value 1N4148WS -> SS54; device Discrete:D'0805' -> diode:DIODE-DO-214AC
- R32: value 12R -> 3R3
- R57: value NC -> 10K
- RST: value BUTTON -> TS24CA; device MySMD:PB157 -> sale:TS24CA
Connections:
- removed net N$13: C19.1, Q1.2, U3.OSCO
- removed net N$15: Q5.D, R24.1
- removed net N$16: C15.2, C17.2, R2.1
- removed net N$20: BT1.2, R24.2
- removed net N$25: R49.2, R52.1, U8.A0
- removed net N$4: C18.1, Q1.1, U3.OSCI
- removed net N$5: Q2.G, R45.2, R50.1
- removed net N$8: LED1.+, R18.1
- removed net N$9: LED1.-, Q2.D
- removed net VRTC: C14.2, C25.2, D5.-, Q5.S, R2.2, U3.VDD
- net 3.3V: no longer C29.2, C30.2, C31.1, C32.1, D5.+, Q5.G, R17.1, R52.2, U8.VDD
- net 5V: now also D3.A, D5.C; no longer D2.-, D3.+, R18.2
- net GND: now also BOOT.1, BOOT.3, BOOT.4, M1.P$1, M2.P$1, M3.P$1, M4.P$1, M5.P$1, M6.P$1, M7.P$1, M8.P$1, RST.3, RST.4; no longer BT1.1, C14.1, C15.1, C17.1, C18.2, C19.2, C25.1, C29.1, C30.1, C31.2, C32.2, FLASH.1, Q2.S, R17.2, R45.1, R49.1, U3.VSS, U8.GND
- net IO0: now also BOOT.2; no longer FLASH.2
- net IO17/I2C_SDA: no longer U3.SDA, U8.SDA
- net IO18/I2C_SCL: no longer U3.SCL, U8.SCL
- net IO38: no longer U8.PENIRQ
- net TXD/IO43: no longer R50.2
- net VBUS: now also D5.A; no longer D2.+
- net VPWR: now also D3.C; no longer D3.-
- net XN: no longer U8.XN
- net XP: no longer U8.XP
- net YN: no longer U8.YN
- net YP: no longer U8.YP
Other:
- note added: "15dB"
- note added: "ESP32-S3 Parallel TFT with Touch 4.3" V3.1"
- note removed: "1V~5.5V"
- note removed: "9dB"
- note removed: "ESP32-S3 Parallel TFT with Touch 4.3“ V2.0"
- note removed: "LED"
- note removed: "NS2009"
